File: Hephaestus v1/Hephaestus v1_5.sch (EAGLE design)
At the start: 42 parts, among them IC1 NC7SZ14P5X, IC3 NC7SZ14P5X

Commit message: Hopefully the resistors and capacitors are up to spec and I can move on.
Parts:
- D5: device diode:DIODE-DO-214AC -> diode:DIODE-DO214AC
- R1, R12, R13, R2, R3, R4, R5, R6, R7, R8, R9: device resistor:R-US_R2512 -> rcl:R-US_R0603
- U$6: value MCP6L02 -> (none)
Connections:
- net GND: now also U$1.THERM_GND
Other:
- note added: "zener"
Changed lines of the file:
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@@
 <part name="SUPPLY1" library="CP-Symbols" deviceset="GND" device=""/>
 <part name="SUPPLY2" library="CP-Symbols" deviceset="GND" device=""/>
-<part name="R6" library="resistor" deviceset="R-US_" device="R2512" value="5k"/>
+<part name="R6" library="rcl" deviceset="R-US_" device="R0603" value="5k"/>
 <part name="U$7" library="CP-Symbols" deviceset="PP5V" device=""/>
 <part name="CART_VOLT_RVP" library="CP-Symbols" deviceset="PP12V_2" device="" value="PP12V_BAT_RP"/>
@@
 <part name="SUPPLY7" library="CP-Symbols" deviceset="GND" device=""/>
 <part name="SUPPLY8" library="CP-Symbols" deviceset="PP12V_2" device="" value="PP12V_BAT"/>
-<part name="R1" library="resistor" deviceset="R-US_" device="R2512" value="100"/>
-<part name="R2" library="resistor" deviceset="R-US_" device="R2512" value="100"/>
-<part name="R3" library="resistor" deviceset="R-US_" device="R2512" value="100"/>
-<part name="R4" library="resistor" deviceset="R-US_" device="R2512" value="100"/>
+<part name="R1" library="rcl" deviceset="R-US_" device="R0603" value="100"/>
+<part name="R2" library="rcl" deviceset="R-US_" device="R0603" value="100"/>
+<part name="R3" library="rcl" deviceset="R-US_" device="R0603" value="100"/>
+<part name="R4" library="rcl" deviceset="R-US_" device="R0603" value="100"/>
 <part name="SUPPLY9" library="CP-Symbols" deviceset="GND" device=""/>
 <part name="U$12" library="CP-Symbols" deviceset="PP5V" device=""/>
@@
 <part name="SUPPLY15" library="CP-Symbols" deviceset="PP12V_2" device="" value="PP12V_BAT_RP"/>
 <part name="IC1" library="74xx-little-de" deviceset="NC7SZ14" device="P5X"/>
-<part name="R5" library="resistor" deviceset="R-US_" device="R2512" value="33k"/>
-<part name="R7" library="resistor" deviceset="R-US_" device="R2512" value="10k"/>
-<part name="D5" library="diode" deviceset="DIODE-" device="DO-214AC" value="12V"/>
+<part name="R5" library="rcl" deviceset="R-US_" device="R0603" value="33k"/>
+<part name="R7" library="rcl" deviceset="R-US_" device="R0603" value="10k"/>
+<part name="D5" library="diode" deviceset="DIODE-" device="DO214AC" value="12V"/>
 <part name="C9" library="eagle-ltspice" deviceset="C" device="C0603" value="1 uF"/>
 <part name="C3" library="eagle-ltspice" deviceset="C" device="C0603" value="1 uF"/>
@@
 <part name="U$21" library="CP-Symbols" deviceset="PP5V" device=""/>
 <part name="SUPPLY31" library="CP-Symbols" deviceset="GND" device=""/>
-<part name="R8" library="resistor" deviceset="R-US_" device="R2512" value="5k"/>
-<part name="R9" library="resistor" deviceset="R-US_" device="R2512" value="5k"/>
+<part name="R8" library="rcl" deviceset="R-US_" device="R0603" value="5k"/>
+<part name="R9" library="rcl" deviceset="R-US_" device="R0603" value="5k"/>
 <part name="SUPPLY17" library="CP-Symbols" deviceset="GND" device=""/>
 <part name="U$6" library="heph_custom_comp" deviceset="MCP6L02" device=""/>
-<part name="R12" library="resistor" deviceset="R-US_" device="R2512" value="5k"/>
-<part name="R13" library="resistor" deviceset="R-US_" device="R2512" value="5k"/>
+<part name="R12" library="rcl" deviceset="R-US_" device="R0603" value="5k"/>
+<part name="R13" library="rcl" deviceset="R-US_" device="R0603" value="5k"/>
 <part name="SUPPLY20" library="CP-Symbols" deviceset="GND" device=""/>
 <part name="U$22" library="CP-Symbols" deviceset="PP5V" device=""/>
@@
 <part name="SUPPLY28" library="CP-Symbols" deviceset="GND" device=""/>
 <part name="C4" library="eagle-ltspice" deviceset="C" device="C0603" value="4.7 uF"/>
+<part name="SUPPLY19" library="CP-Symbols" deviceset="GND" device=""/>
 </parts>
 <sheets>
@@
 <text x="81.28" y="20.32" size="7.62" layer="90">UPDATE BRAKING H-BRIDGE</text>
 <text x="99.06" y="5.08" size="5.08" layer="94">Braking H-Bridge</text>
+<text x="-17.78" y="58.42" size="1.778" layer="97">zener</text>
 </plain>
 <instances>
@@
 <instance part="SUPPLY28" gate="G$1" x="381" y="170.18"/>
 <instance part="C4" gate="G$1" x="381" y="175.26" rot="R180"/>
+<instance part="SUPPLY19" gate="G$1" x="137.16" y="137.16"/>
 </instances>
 <busses>
@@
 <wire x1="381" y1="172.72" x2="381" y2="170.18" width="0.1524" layer="91"/>
 </segment>
+<segment>
+<pinref part="U$1" gate="G$1" pin="THERM_GND"/>
+<pinref part="SUPPLY19" gate="G$1" pin="GND"/>
+<wire x1="139.7" y1="137.16" x2="137.16" y2="137.16" width="0.1524" layer="91"/>
+</segment>
 </net>

Commit message: Most recent changes (gate logic, decoupling capacitors, everything hopefully properly specced) hopefully
Parts:
- added C10, C11: 22 uF, eagle-ltspice:CC0603
- C2: value 22 uF -> 47 uF
Connections:
- net GND: now also C10.1, C11.1
- net MCU_DIR_S: now also U$1.AHI; no longer U$1.BLO
- net MCU_DIR_S_INV: now also U$1.BHI; no longer U$1.ALO
- net MCU_PWM_S: now also U$1.ALO; no longer U$1.AHI
- net MCU_PWM_S_INV: now also U$1.BLO; no longer U$1.BHI
- net PP12V_2: now also C10.2, C11.2
Changed lines of the file:
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@@
 <part name="D3" library="heph_custom_comp" deviceset="PMEG6020ETR" device="" value="PMEG6020ETR"/>
 <part name="D4" library="heph_custom_comp" deviceset="PMEG6020ETR" device="" value="PMEG6020ETR"/>
-<part name="C2" library="eagle-ltspice" deviceset="C" device="C0603" value="22 uF"/>
+<part name="C2" library="eagle-ltspice" deviceset="C" device="C0603" value="47 uF"/>
 <part name="SUPPLY6" library="CP-Symbols" deviceset="GND" device=""/>
 <part name="CART_VOLT_RVP1" library="CP-Symbols" deviceset="PP12V_2" device="" value="PP12V_BAT_RP"/>
@@
 <part name="C4" library="eagle-ltspice" deviceset="C" device="C0603" value="4.7 uF"/>
 <part name="SUPPLY19" library="CP-Symbols" deviceset="GND" device=""/>
+<part name="CART_VOLT_RVP2" library="CP-Symbols" deviceset="PP12V_2" device="" value="PP12V_BAT_RP"/>
+<part name="C10" library="eagle-ltspice" deviceset="C" device="C0603" value="22 uF"/>
+<part name="SUPPLY21" library="CP-Symbols" deviceset="GND" device=""/>
+<part name="CART_VOLT_RVP3" library="CP-Symbols" deviceset="PP12V_2" device="" value="PP12V_BAT_RP"/>
+<part name="C11" library="eagle-ltspice" deviceset="C" device="C0603" value="22 uF"/>
+<part name="SUPPLY23" library="CP-Symbols" deviceset="GND" device=""/>
 </parts>
 <sheets>
@@
 <instance part="C4" gate="G$1" x="381" y="175.26" rot="R180"/>
 <instance part="SUPPLY19" gate="G$1" x="137.16" y="137.16"/>
+<instance part="CART_VOLT_RVP2" gate="G$1" x="15.24" y="86.36"/>
+<instance part="C10" gate="G$1" x="15.24" y="76.2" rot="R180"/>
+<instance part="SUPPLY21" gate="G$1" x="15.24" y="71.12"/>
+<instance part="CART_VOLT_RVP3" gate="G$1" x="25.4" y="81.28"/>
+<instance part="C11" gate="G$1" x="25.4" y="71.12" rot="R180"/>
+<instance part="SUPPLY23" gate="G$1" x="25.4" y="66.04"/>
 </instances>
 <busses>
@@
 </segment>
 <segment>
-<pinref part="U$1" gate="G$1" pin="AHI"/>
-<wire x1="170.18" y1="154.94" x2="177.8" y2="154.94" width="0.1524" layer="91"/>
-<label x="177.8" y="154.94" size="1.016" layer="95" xref="yes"/>
+<pinref part="U$1" gate="G$1" pin="ALO"/>
+<wire x1="170.18" y1="157.48" x2="177.8" y2="157.48" width="0.1524" layer="91"/>
+<label x="177.8" y="157.48" size="1.016" layer="95" xref="yes"/>
 </segment>
 </net>
@@
 <wire x1="139.7" y1="137.16" x2="137.16" y2="137.16" width="0.1524" layer="91"/>
 </segment>
+<segment>
+<pinref part="C10" gate="G$1" pin="1"/>
+<pinref part="SUPPLY21" gate="G$1" pin="GND"/>
+<wire x1="15.24" y1="73.66" x2="15.24" y2="71.12" width="0.1524" layer="91"/>
+</segment>
+<segment>
+<pinref part="C11" gate="G$1" pin="1"/>
+<pinref part="SUPPLY23" gate="G$1" pin="GND"/>
+<wire x1="25.4" y1="68.58" x2="25.4" y2="66.04" width="0.1524" layer="91"/>
+</segment>
 </net>
 <net name="I2C_SCL" class="0">
@@
 <wire x1="304.8" y1="76.2" x2="307.34" y2="76.2" width="0.1524" layer="91"/>
 </segment>
+<segment>
+<pinref part="C10" gate="G$1" pin="2"/>
+<pinref part="CART_VOLT_RVP2" gate="G$1" pin="PP12V_2"/>
+<wire x1="15.24" y1="81.28" x2="15.24" y2="83.82" width="0.1524" layer="91"/>
+</segment>
+<segment>
+<pinref part="C11" gate="G$1" pin="2"/>
+<pinref part="CART_VOLT_RVP3" gate="G$1" pin="PP12V_2"/>
+<wire x1="25.4" y1="76.2" x2="25.4" y2="78.74" width="0.1524" layer="91"/>
+</segment>
 </net>
 <net name="PP5V" class="0">
@@
 </segment>
 <segment>
-<pinref part="U$1" gate="G$1" pin="BLO"/>
-<wire x1="170.18" y1="162.56" x2="177.8" y2="162.56" width="0.1524" layer="91"/>
-<label x="177.8" y="162.56" size="1.016" layer="95" xref="yes"/>
-</segment>
-<segment>
 <pinref part="IC1" gate="G$1" pin="I"/>
 <wire x1="129.54" y1="111.76" x2="132.08" y2="111.76" width="0.1524" layer="91"/>
 <label x="132.08" y="111.76" size="1.016" layer="95" xref="yes"/>
+</segment>
+<segment>
+<pinref part="U$1" gate="G$1" pin="AHI"/>
+<wire x1="170.18" y1="154.94" x2="177.8" y2="154.94" width="0.1524" layer="91"/>
+<label x="177.8" y="154.94" size="1.016" layer="95" xref="yes"/>
 </segment>
 </net>
@@
 </segment>
 <segment>
-<pinref part="U$1" gate="G$1" pin="ALO"/>
-<wire x1="177.8" y1="157.48" x2="170.18" y2="157.48" width="0.1524" layer="91"/>
-<label x="177.8" y="157.48" size="1.016" layer="95" xref="yes"/>
+<pinref part="U$1" gate="G$1" pin="BHI"/>
+<wire x1="170.18" y1="160.02" x2="177.8" y2="160.02" width="0.1524" layer="91"/>
+<label x="177.8" y="160.02" size="1.016" layer="95" xref="yes"/>
 </segment>
 </net>
@@
 </segment>
 <segment>
-<pinref part="U$1" gate="G$1" pin="BHI"/>
-<wire x1="170.18" y1="160.02" x2="177.8" y2="160.02" width="0.1524" layer="91"/>
-<label x="177.8" y="160.02" size="1.016" layer="95" xref="yes"/>
-</segment>
-</net>
+<label x="177.8" y="162.56" size="1.016" layer="95" xref="yes"/>
+<pinref part="U$1" gate="G$1" pin="BLO"/>
+<wire x1="170.18" y1="162.56" x2="177.8" y2="162.56" width="0.1524" layer="91"/>
+<label x="177.8" y="162.56" size="1.016" layer="95" xref="yes"/>
+</segment>
+</net>
